Commit message: 'Fixed' gravity issue. Seems related to update rate of motor plugin

File: src/roberto_models_jade/models/inertia_tensors.xacro (robot description, xacro)
@@ -3,5 +3,5 @@
   see https://github.com/uos/uos_tools/blob/fuerte/uos_common_urdf/common.xacro and
   see http://answers.gazebosim.org/question/4372/the-inertia-matrix-explained/ -->
-<robot xmlns:xacro="http://ros.org/wiki/xacro">
+<robot xmlns:xacro="http://www.ros.org/wiki/xacro">
   <xacro:property name="M_PI" value="3.1415926535897931" />
   <!-- see https://secure.wikimedia.org/wikipedia/en/wiki/List_of_moment_of_inertia_tensors -->

File: src/roberto_models_jade/models/platform/roberto.xacro (robot description, xacro)
@@ -1,18 +1,17 @@
 <?xml version="1.0"?>
-<robot xmlns:xacro="http://ros.org/wiki/xacro" name="roberto" >
-    <xacro:arg name="model_dir" default="$(find roberto_models)/models/platform"/>
+<robot xmlns:xacro="http://www.ros.org/wiki/xacro" name="roberto" >
+    <xacro:arg name="model_dir" default="$(find roberto_models_jade)/models/platform"/>
     <!-- Import colors (for Rviz)-->
-    <xacro:include filename="$(find roberto_models)/models/materials.xacro" />
+    <xacro:include filename="$(find roberto_models_jade)/models/materials.xacro" />
     <!-- Import robot -->
     <xacro:property name="model_dir" value="$(arg model_dir)/roberto_body"/>
-    <xacro:include filename="${model_dir}/body.xacro"/>
-    <xacro:RobertoBody name="body" parent="base" mesh_collis="simplified" mesh_visual="detailed"/><!-- simplified detailed empty-->
+    <xacro:include filename="$(find roberto_models_jade)/models/platform/roberto_body/body.xacro"/>
+    <xacro:RobertoBody name="body" parent="base" mesh_collis="simplified" mesh_visual="detailed"/>   <!-- simplified detailed empty-->
     <!-- Import platform plugins -->
-    <xacro:property name="model_dir" value="$(arg model_dir)"/>
-    <xacro:include filename="${model_dir}/roberto_plugins.xacro" />
-    <xacro:RobertoMotorDrivePlugin        />
+    <xacro:include filename="$(find roberto_models_jade)/models/platform/roberto_plugins.gazebo" />
+    <xacro:RobertoMotorDrivePlugin />
     <!-- IMU
-    <xacro:property name="model_dir" value="$(find roberto_models)/models/sensors/imu"/>
-    <xacro:include filename="$(find roberto_models)/models/sensors/imu/imu.xacro"/>
+    <xacro:property name="model_dir" value="$(find roberto_models_jade)/models/sensors/imu"/>
+    <xacro:include filename="$(find roberto_models_jade)/models/sensors/imu/imu.xacro"/>
     <xacro:imu_sensor name="imu9dof" parent="base_link" xyz="0.0 0.05 0.262" rpy="0 0 ${pi/2}"/>-->
     <!-- Camera

File: src/roberto_models_jade/models/platform/roberto_body/body.xacro (robot description, xacro)
@@ -6,4 +6,5 @@
 	<xacro:include filename="wheel_mount.xacro"/>
 	<xacro:include filename="wheel.xacro"/>
+	<xacro:include filename="spacer.xacro"/>
 	<xacro:macro name="RobertoBody" params="name parent mesh_collis mesh_visual" >
 		<!-- Base link -->

File: src/roberto_models_jade/models/platform/roberto_body/parameters.xacro (robot description, xacro)
@@ -14,8 +14,8 @@
 	<xacro:property name="frontWheelMass" value="0.045"/>
 	<xacro:property name="rearWheelWidth" value="0.04"/>
-	<xacro:property name="rearWheelMass" value="0.05"/>
+	<xacro:property name="rearWheelMass" value="0.050"/>
 	<xacro:property name="motorMountRadius" value="0.02"/>
 	<xacro:property name="motorMountLength" value="0.07"/>
-	<xacro:property name="motorMountMass" value="0.19"/>
+	<xacro:property name="motorMountMass" value="0.190"/>
 	<xacro:property name="motorMountPos" value="0.085"/>
 	<xacro:property name="spacerRadius" value="0.004"/>
@@ -26,4 +26,6 @@
 	<xacro:property name="spacerPosZ" value="0.079"/>
 	<xacro:property name="cameraSize" value="0.05"/>
-	<xacro:property name="cameraMass" value="0.1"/>
+	<xacro:property name="cameraMass" value="0.100"/>
+	<xacro:property name="servoLowerLimit" value="0.2618" />
+    <xacro:property name="servoUpperLimit" value="1.57" />
 </robot>

File: src/roberto_models_jade/models/platform/roberto_body/platform_bottom.xacro (robot description, xacro)
@@ -1,7 +1,7 @@
 <?xml version="1.0"?>
 <robot xmlns:xacro="http://www.ros.org/wiki/xacro">
-	<xacro:include filename="$(find roberto_models)/models/inertia_tensors.xacro"/>
+	<xacro:include filename="$(find roberto_models_jade)/models/inertia_tensors.xacro"/>
 	<xacro:macro name="RobertoPlatformBottom" params="name parent mesh_collis:=^|simplified mesh_visual:=^|detailed model_dir:=^">
-		<xacro:property name="ParrentLink2ThisLink"> <!--parrent link to this joint tf-->
+		<xacro:property name="ParentLink2ThisLink"> <!--parent link to this joint tf-->
 			<origin xyz="0 0 0" rpy="0 0 0"/>
 	    </xacro:property>
@@ -30,5 +30,5 @@
 			<parent link="${parent}_link"/>
 			<child  link="${name}_link" />
-			<xacro:insert_block name="ParrentLink2ThisLink" />
+			<xacro:insert_block name="ParentLink2ThisLink" />
 	    </joint>
 	    <link name="${name}_link">
@@ -37,27 +37,7 @@
 			<collision> <xacro:insert_block name="ThisCollis"/> </collision>
 	    </link>
-	    <!--
 	    <gazebo reference="${name}_link">
-			<material>Gazebo/LightBlueLaser</material>
-			<selfCollide>false</selfCollide>
+			<!--<material>Gazebo/LightBlueLaser</material> -->
 	    </gazebo>
-		-->
-		<link name="platform_top">
-			<visual>
-			  	<geometry>
-			    	<mesh filename="package://roberto_description/meshes/platform_top.dae"/>
-			  	</geometry>
-			  	<origin rpy="0 ${PI} 0" xyz="0.02 -0.03 0"/>
-			</visual>
-			<!--<collision>
-				<geometry>
-					<box size="${platformTopLength} ${platformTopWidth} ${platformTopHeight}"/>
-				</geometry>
-				<origin rpy="0 ${PI} 0" xyz="0 0 0"/>
-			</collision>-->
-			<inertial>
-				<mass value="${platformTopMass}"/>
-				<xacro:box_inertia m="${platformTopMass}" x="${platformTopLength}" y="${platformTopWidth}" z="${platformTopHeight}"/>
-			</inertial>
-		</link>
 	</xacro:macro>
+</robot>

File: src/roberto_models_jade/models/platform/roberto_body/platform_top.xacro (robot description, xacro)
@@ -1,8 +1,8 @@
 <?xml version="1.0"?>
 <robot xmlns:xacro="http://www.ros.org/wiki/xacro">
-	<xacro:include filename="$(find roberto_models)/models/inertia_tensors.xacro"/>
+	<xacro:include filename="$(find roberto_models_jade)/models/inertia_tensors.xacro"/>
 	<xacro:macro name="RobertoPlatformTop" params="name parent mesh_collis:=^|simplified mesh_visual:=^|detailed model_dir:=^">
-		<xacro:property name="ParrentLink2ThisLink"> <!--parrent link to this joint tf-->
-			<origin xyz="0 0 0" rpy="0 0 0"/>
+		<xacro:property name="ParentLink2ThisLink"> <!--parent link to this joint tf-->
+			<origin xyz="-0.01 0.03 ${spacerLength+spacerPosZ-platformTopHeight-0.001}" rpy="0 0 0"/>
 	    </xacro:property>
 	    <xacro:property name="ThisLink2Inert"> <!--this link 2 inertial center tf, mass data-->
@@ -10,10 +10,10 @@
 	    </xacro:property>
 	    <xacro:property name="ThisLink2STL"> <!--this link 2 mesh center tf, file-->
-			<origin xyz="0.02 -0.03 0" rpy="0 ${pi} 0"/>
+			<origin xyz="${platformTopLength/2} -${platformTopWidth/2} 0" rpy="0 ${pi} 0"/>
 			<geometry> <mesh filename="file://${model_dir}/meshes/platform_top.dae"/> </geometry>
 			<!--<material name="light_blue"/> -->
 	    </xacro:property>
 	    <xacro:property name="ThisLink2XML"> <!--this link 2 simple mesh center tf, file-->
-			<origin xyz="0 0 0.06" rpy="0 0 0"/>
+			<origin xyz="0 0 0" rpy="0 ${pi} 0"/>
 			<geometry> <box size="${platformTopLength} ${platformTopWidth} ${platformTopHeight}" /> </geometry>
 			<!--<material name="light_blue"/> -->
@@ -30,5 +30,5 @@
 			<parent link="${parent}_link"/>
 			<child  link="${name}_link" />
-			<xacro:insert_block name="ParrentLink2ThisLink" />
+			<xacro:insert_block name="ParentLink2ThisLink" />
 	    </joint>
 	    <link name="${name}_link">
@@ -37,9 +37,7 @@
 			<collision> <xacro:insert_block name="ThisCollis"/> </collision>
 	    </link>
-	    <!--
 	    <gazebo reference="${name}_link">
-			<material>Gazebo/LightBlueLaser</material>
-			<selfCollide>false</selfCollide>
+			<!--<material>Gazebo/LightBlueLaser</material> -->
 	    </gazebo>
-		-->
 	</xacro:macro>
+</robot>

File: src/roberto_models_jade/models/platform/roberto_body/spacer.xacro (robot description, xacro)
@@ -1,12 +1,12 @@
 <?xml version="1.0"?>
 <robot xmlns:xacro="http://www.ros.org/wiki/xacro">
-  <xacro:include filename="$(find roberto_models)/models/inertia_tensors.xacro"/>
+  <xacro:include filename="$(find roberto_models_jade)/models/inertia_tensors.xacro"/>
   <xacro:macro name="Spacer" params="name parent fb lr mesh_collis:=^|simplified mesh_visual:=^|detailed model_dir:=^">
     <!-- Selecting origin position -->
-    <xacro:property name="tX">1</xacro:property>
-    <xacro:property name="tY">1</xacro:property>
-    <xacro:if value="${fb ==   'B'}"> <xacro:property name="tY">-1</xacro:property> </xacro:if>
-    <xacro:if value="${lr ==   'L'}"> <xacro:property name="tX">-1</xacro:property> </xacro:if>
-    <xacro:property name="ParrentLink2ThisLink"> <!--parrent link to this joint tf-->
+    <xacro:property name="tX" value="1" />
+    <xacro:property name="tY" value="1" />
+    <xacro:if value="${fb ==   'B'}"> <xacro:property name="tY" value="-1" /> </xacro:if>
+    <xacro:if value="${lr ==   'L'}"> <xacro:property name="tX" value="-1" /> </xacro:if>
+    <xacro:property name="ParentLink2ThisLink"> <!--parent link to this joint tf-->
       <axis xyz="0 0 1"/>
       <origin xyz="${spacerPosX*tX} ${spacerPosY*tY} ${spacerPosZ}" rpy="0 0 0" />
@@ -36,5 +36,5 @@
       <parent link="${parent}_link"/>
       <child  link="${name}${fb}${lr}_link" />
-      <xacro:insert_block name="ParrentLink2ThisLink" />
+      <xacro:insert_block name="ParentLink2ThisLink" />
     </joint>
     <link name="${name}${fb}${lr}_link">

File: src/roberto_models_jade/models/platform/roberto_body/wheel.xacro (robot description, xacro)
@@ -1,17 +1,18 @@
 <?xml version="1.0"?>
 <robot xmlns:xacro="http://www.ros.org/wiki/xacro">
-  <xacro:include filename="$(find roberto_models)/models/inertia_tensors.xacro"/>
+  <xacro:include filename="$(find roberto_models_jade)/models/inertia_tensors.xacro"/>
   <xacro:macro name="Wheel" params="name parent fb lr mesh_collis:=^|simplified mesh_visual:=^|detailed model_dir:=^">
     <!-- Selecting origin position -->
     <xacro:property name="mass" value="${frontWheelMass}" />
     <xacro:property name="width" value="${frontWheelWidth}" />
-    <xacro:property name="tY">1</xacro:property>
-    <xacro:if value="${lr ==   'L'}"> <xacro:property name="tY">-1</xacro:property> </xacro:if>
+    <xacro:property name="tY" value="1" />
+    <xacro:if value="${lr ==   'L'}"> <xacro:property name="tY" value="-1" /> </xacro:if>
     <xacro:if value="${fb ==   'B'}"> <xacro:property name="mass" value="${rearWheelMass}" /> <xacro:property name="width" value="${rearWheelWidth}" /> </xacro:if>
-    <xacro:property name="ParrentLink2ThisLink"> <!--parrent link to this joint tf-->
+    <xacro:property name="ParentLink2ThisLink"> <!--parent link to this joint tf-->
       <origin xyz="${wheelPos*tY} 0 0" rpy="0 0 0" />
       <axis xyz="1 0 0" rpy="0 0 0" />
-      <limit effort="10" velocity="4"/>
-      <joint_properties damping="0.0" friction="0.0"/>
+      <!--<dynamics damping="0.7" />-->
+      <!--<limit effort="10" velocity="4"/>
+      <joint_properties damping="0.0" friction="0.0"/>-->
     </xacro:property>
     <xacro:property name="ThisLink2Inert"> <!--this link 2 inertial center tf, mass data-->
@@ -39,5 +40,5 @@
       <parent link="${parent}${fb}${lr}_link"/>
       <child  link="${name}${fb}${lr}_link" />
-      <xacro:insert_block name="ParrentLink2ThisLink" />
+      <xacro:insert_block name="ParentLink2ThisLink" />
     </joint>
     <link name="${name}${fb}${lr}_link">
@@ -47,10 +48,11 @@
     </link>
     <gazebo reference="${name}${fb}${lr}_link">
-      <mu1 value="5.9"/>
-      <mu2 value="5.9"/>
-      <kp value="1000000.0"/>
-      <kd value="10"/>
+      <!--<selfCollide>false</selfCollide>-->
+      <mu1>5.9</mu1>
+      <kp>1000000.0</kp>
+      <kd>100.0</kd>
+      <minDepth>0.001</minDepth>
+      <maxVel>1.0</maxVel>
       <material>Gazebo/Black</material>
-      <selfCollide>false</selfCollide>
     </gazebo>
   </xacro:macro>

File: src/roberto_models_jade/models/platform/roberto_body/wheel_mount.xacro (robot description, xacro)
@@ -1,25 +1,26 @@
 <?xml version="1.0"?>
 <robot xmlns:xacro="http://www.ros.org/wiki/xacro">
-  <xacro:include filename="$(find roberto_models)/models/inertia_tensors.xacro"/>
+  <xacro:include filename="$(find roberto_models_jade)/models/inertia_tensors.xacro"/>
   <xacro:macro name="WheelMount" params="name parent fb lr mesh_collis:=^|simplified mesh_visual:=^|detailed model_dir:=^">
     <!-- Selecting origin position -->
-    <xacro:property name="adjust">0</xacro:property>
-    <xacro:property name="tX">1</xacro:property>
-    <xacro:property name="tY">1</xacro:property>
-    <xacro:if value="${lr ==   'L'}"> <xacro:property name="tX">-1</xacro:property> </xacro:if>
-    <xacro:if value="${fb ==   'B'}"> <xacro:property name="adjust" value="0.01" /> </xacro:if>
+    <xacro:property name="adjust" value="0" />
+    <xacro:property name="tX" value="1" />
+    <xacro:property name="tY" value="1" />
+    <xacro:if value="${lr == 'L'}"> <xacro:property name="tX" value="-1" /> </xacro:if>
+    <xacro:if value="${fb == 'B'}"> <xacro:property name="tY" value="-1" /> <xacro:property name="adjust" value="0.01" /> </xacro:if>
     <!-- Select servo limits -->
     <xacro:property name="ll" value="${servoLowerLimit}"/>
     <xacro:property name="ul" value="${servoUpperLimit}"/>
-    <xacro:if value="${fb ==   'B' and lr == 'L'}"> <xacro:property name="ll" value="-${servoLowerLimit}" /> <xacro:property name="ul" value="${servoUpperLimit}" /> </xacro:if>
-    <xacro:if value="${fb ==   'B' and lr == 'R'}"> <xacro:property name="ll" value="-${servoUpperLimit}" /> <xacro:property name="ul" value="${servoLowerLimit}" /> </xacro:if>
-    <xacro:if value="${fb ==   'F' and lr == 'L'}"> <xacro:property name="ll" value="-${servoUpperLimit}" /> <xacro:property name="ul" value="${servoLowerLimit}" /> </xacro:if>
-    <xacro:if value="${fb ==   'F' and lr == 'R'}"> <xacro:property name="ll" value="-${servoLowerLimit}" /> <xacro:property name="ul" value="${servoUpperLimit}" /> </xacro:if>
-    <xacro:property name="ParrentLink2ThisLink"> <!--parrent link to this joint tf-->
+    <xacro:if value="${fb == 'B' and lr == 'L'}"> <xacro:property name="ll" value="-${servoLowerLimit}" /> <xacro:property name="ul" value="${servoUpperLimit}" /> </xacro:if>
+    <xacro:if value="${fb == 'B' and lr == 'R'}"> <xacro:property name="ll" value="-${servoUpperLimit}" /> <xacro:property name="ul" value="${servoLowerLimit}" /> </xacro:if>
+    <xacro:if value="${fb == 'F' and lr == 'L'}"> <xacro:property name="ll" value="-${servoUpperLimit}" /> <xacro:property name="ul" value="${servoLowerLimit}" /> </xacro:if>
+    <xacro:if value="${fb == 'F' and lr == 'R'}"> <xacro:property name="ll" value="-${servoLowerLimit}" /> <xacro:property name="ul" value="${servoUpperLimit}" /> </xacro:if>
+    <xacro:property name="ParentLink2ThisLink"> <!--parent link to this joint tf-->
       <origin xyz="${motorMountPos*tX} ${motorMountPos*tY} ${wheelRadius}" rpy="0 0 0" />
       <axis xyz="0 0 1" rpy="0 0 0" />
-      <limit effort="1000.0" velocity="4" lower="${ll}" upper="${ul}"/>
-      <origin xyz="${wheelPos*tY} 0 0" rpy="0 0 0" />
-      <limit effort="10" velocity="4"/>
+      <limit effort="10.0" velocity="4" lower="${ll}" upper="${ul}"/>
+      <!--<dynamics damping="0.7" />-->
+      <!--<origin xyz="${wheelPos*tY} 0 0" rpy="0 0 0" />
+      <limit effort="10" velocity="4"/>-->
     </xacro:property>
     <xacro:property name="ThisLink2Inert"> <!--this link 2 inertial center tf, mass data-->
@@ -27,5 +28,5 @@
     </xacro:property>
     <xacro:property name="ThisLink2STL"> <!--this link 2 mesh center tf, file-->
-      <origin xyz="0.02 -0.03 0" rpy="0 ${pi/2} 0"/>
+      <origin xyz="0 0 0" rpy="0 ${pi/2} 0"/>
       <geometry> <mesh filename="file://${model_dir}/meshes/platform_top.dae"/> </geometry>
       <material name="grey"/>
@@ -44,8 +45,8 @@
     <xacro:if value="${mesh_collis == 'simplified'}"> <xacro:property name="ThisCollis">  <xacro:insert_block name="ThisLink2XML"/> </xacro:property> </xacro:if><!--minimalist mesh-->
     <!-- joint and link definition -->
-    <joint name="${parent}2${name}${fb}${lr}_joint" type="continuous">
+    <joint name="${parent}2${name}${fb}${lr}_joint" type="revolute">
       <parent link="${parent}_link"/>
       <child  link="${name}${fb}${lr}_link" />
-      <xacro:insert_block name="ParrentLink2ThisLink" />
+      <xacro:insert_block name="ParentLink2ThisLink" />
     </joint>
     <link name="${name}${fb}${lr}_link">
@@ -55,10 +56,11 @@
     </link>
     <gazebo reference="${name}${fb}${lr}_link">
-      <mu1 value="5.9"/>
-      <mu2 value="5.9"/>
-      <kp value="1000000.0"/>
-      <kd value="10"/>
+      <mu1>5.9</mu1>
+      <mu2>5.9</mu2>
+      <kp>1000000.0</kp>
+      <kd>100.0</kd>
+      <minDepth>0.001</minDepth>
+      <maxVel>1.0</maxVel>
       <material>Gazebo/Grey</material>
-      <selfCollide>false</selfCollide>
     </gazebo>
   </xacro:macro>
