Commit message: Fixed issue with motorplugin, by implementing PID control

File: src/roberto_models_jade/models/platform/roberto.xacro (robot description, xacro)
@@ -15,7 +15,6 @@
     <xacro:include filename="$(find roberto_models_jade)/models/sensors/imu/imu.xacro"/>
     <xacro:imu_sensor name="imu9dof" parent="base_link" xyz="0.0 0.05 0.262" rpy="0 0 ${pi/2}"/>-->
-    <!-- Camera
-    <xacro:include filename="$(find blue_gazebo)/xacro/camera/camera.xacro"/>
-    <xacro:cam name="front_camera" parent="body" xyz="0 0 0.5" rpy="0 0 ${pi/2}"/>
-    -->
+    <!-- Camera -->
+    <xacro:include filename="$(find roberto_models_jade)/models/sensors/camera/camera.xacro"/>
+    <xacro:cam name="front_camera" parent="body_top" angle="${M_PI/10}" xyz="0 0.01 0.0375" rpy="0 0 ${M_PI/2}"/>
 </robot>

File: src/roberto_models_jade/models/platform/roberto_body/parameters.xacro (robot description, xacro)
@@ -6,6 +6,6 @@
 	<xacro:property name="platformMass" value="0.200"/>
 	<xacro:property name="platformTopHeight" value="0.005"/>
-	<xacro:property name="platformTopLength" value="0.200"/>
-	<xacro:property name="platformTopWidth" value="0.200"/>
+	<xacro:property name="platformTopLength" value="0.160"/>
+	<xacro:property name="platformTopWidth" value="0.180"/>
 	<xacro:property name="platformTopMass" value="0.125"/>
 	<xacro:property name="wheelRadius" value="0.04"/>
@@ -25,5 +25,4 @@
 	<xacro:property name="spacerPosY" value="0.052"/>
 	<xacro:property name="spacerPosZ" value="0.079"/>
-	<xacro:property name="cameraSize" value="0.05"/>
 	<xacro:property name="cameraMass" value="0.100"/>
 	<xacro:property name="servoLowerLimit" value="0.2618" />

File: src/roberto_models_jade/models/platform/roberto_body/platform_top.xacro (robot description, xacro)
@@ -4,11 +4,11 @@
 	<xacro:macro name="RobertoPlatformTop" params="name parent mesh_collis:=^|simplified mesh_visual:=^|detailed model_dir:=^">
 		<xacro:property name="ParentLink2ThisLink"> <!--parent link to this joint tf-->
-			<origin xyz="-0.01 0.03 ${spacerLength+spacerPosZ-platformTopHeight-0.001}" rpy="0 0 0"/>
+			<origin xyz="0 0 ${spacerLength+spacerPosZ-platformTopHeight-0.001}" rpy="0 0 0"/>
 	    </xacro:property>
 	    <xacro:property name="ThisLink2Inert"> <!--this link 2 inertial center tf, mass data-->
-			<box_inertial x="${platformTopLength}" y="${platformTopWidth}"  z="${platformTopHeight}" mass="${platformTopMass}" />
+			<box_inertial x="${platformTopWidth}" y="${platformTopLength}"  z="${platformTopHeight}" mass="${platformTopMass}" />
 	    </xacro:property>
 	    <xacro:property name="ThisLink2STL"> <!--this link 2 mesh center tf, file-->
-			<origin xyz="${platformTopLength/2} -${platformTopWidth/2} 0" rpy="0 ${pi} 0"/>
+			<origin xyz="${platformTopWidth/2} -${platformTopLength/2} 0" rpy="0 ${pi} 0"/>
 			<geometry> <mesh filename="file://${model_dir}/meshes/platform_top.dae"/> </geometry>
 			<!--<material name="light_blue"/> -->
@@ -16,5 +16,5 @@
 	    <xacro:property name="ThisLink2XML"> <!--this link 2 simple mesh center tf, file-->
 			<origin xyz="0 0 0" rpy="0 ${pi} 0"/>
-			<geometry> <box size="${platformTopLength} ${platformTopWidth} ${platformTopHeight}" /> </geometry>
+			<geometry> <box size="${platformTopWidth} ${platformTopLength} ${platformTopHeight}" /> </geometry>
 			<!--<material name="light_blue"/> -->
 	    </xacro:property>

Commit message: Added working IMU to jade model

File: src/roberto_models_jade/models/platform/roberto.xacro (robot description, xacro)
@@ -11,8 +11,8 @@
     <xacro:include filename="$(find roberto_models_jade)/models/platform/roberto_plugins.gazebo" />
     <xacro:RobertoMotorDrivePlugin />
-    <!-- IMU
-    <xacro:property name="model_dir" value="$(find roberto_models_jade)/models/sensors/imu"/>
-    <xacro:include filename="$(find roberto_models_jade)/models/sensors/imu/imu.xacro"/>
-    <xacro:imu_sensor name="imu9dof" parent="base_link" xyz="0.0 0.05 0.262" rpy="0 0 ${pi/2}"/>-->
+    <!-- IMU -->
+    <xacro:property name="model_dir" value="$(find roberto_models_jade)/models/sensors/IMU"/>
+    <xacro:include filename="$(find roberto_models_jade)/models/sensors/IMU/imu.xacro"/>
+    <xacro:imu_sensor name="imu9dof" parent="body_link" xyz="0.0 0.0 0.0685" rpy="0 0 0"/>
     <!-- Camera -->
     <xacro:include filename="$(find roberto_models_jade)/models/sensors/camera/camera.xacro"/>

File: src/roberto_models_jade/models/sensors/IMU/imu.xacro (robot description, xacro)
@@ -1,5 +1,4 @@
 <?xml version="1.0"?>
 <robot xmlns:xacro="http://www.ros.org/wiki/xacro">
-<!-- Front Laser -->
 <xacro:macro name="imu_sensor" params="name parent xyz rpy model_dir:=^" >
     <joint name="${parent}_${name}_joint" type="fixed">
@@ -11,17 +10,17 @@
     <link name="${name}">
       <collision>
-        <origin xyz="0 0 0.0015" rpy="0 0 0"/>
+        <origin xyz="0 0 0" rpy="0 0 0"/>
         <geometry>
-          <box size="0.004 0.003 0.003"/>
+          <box size="0.003 0.003 0.001"/>
         </geometry>
       </collision>
       <visual>
-        <origin xyz="0 0 -0.025" rpy="0 0 ${-M_PI/2}"/>
+        <origin xyz="0 0 0" rpy="0 0 0"/>
         <geometry>
-          <mesh filename="file://$(find tuw_gazebo_models)/models/sensors/imu/meshes/imu_razor_9DOF.dae" scale="0.001 0.001 0.001"/>
+          <box size="0.003 0.003 0.001" />
         </geometry>
       </visual>
       <inertial>
-        <mass value="1e-5" />
+        <mass value="1e-6" />
         <origin xyz="0 0 0" rpy="0 0 0"/>
         <inertia ixx="1e-9" ixy="0" ixz="0" iyy="1e-9" iyz="0" izz="1e-9" />
@@ -59,5 +58,5 @@
     </xacro:property>
     <gazebo>
-	<plugin name="gazebo_ros_imu9dof" filename="libtuw_gazebo_ros_imu9dof.so" >
+	<plugin name="gazebo_ros_imu9dof" filename="libroberto_gazebo_ros_imu9dof.so" >
 	    <rosDebugLevel>Debug</rosDebugLevel>
 	    <robotNamespace></robotNamespace>

File: src/roberto_models_jade/models/sensors/TOF/tof.xacro (robot description, xacro)
@@ -39,13 +39,12 @@
 		<scan>
 		    <horizontal>
-			<!-- The RPLidar has 360 steps with 1 Degree resolution -->
 			<resolution>1</resolution>
-			<samples>360</samples> <min_angle>-3.141592</min_angle> <max_angle>3.124139361</max_angle> <!-- -180 to 180 Degree -->
+			<samples>1</samples> <min_angle>0</min_angle> <max_angle>0</max_angle>
 		    </horizontal>
 		</scan>
 		<range>
 		    <min>0.04</min>
-		    <max>6</max>
-		    <resolution>0.02</resolution>
+		    <max>2</max>
+		    <resolution>0.01</resolution>
 		</range>
 		<noise>
@@ -56,9 +55,9 @@
 	    </ray>
 	    <plugin name="gazebo_ros_laser_RPLidar_driver" filename="${driver_type}" >
-		<rosDebugLevel>Debug</rosDebugLevel>
-		<robotNamespace></robotNamespace>
-		<topicName>${frame_names}</topicName>
-		<frameName>${topic_names}</frameName>
-		<rangeMin>0.2</rangeMin>
+			<rosDebugLevel>Debug</rosDebugLevel>
+			<robotNamespace></robotNamespace>
+			<topicName>${frame_names}</topicName>
+			<frameName>${topic_names}</frameName>
+			<rangeMin>0.2</rangeMin>
 	    </plugin>
         </sensor>
