Commit message: Fixed IMU and odom

File: src/roberto_models_jade/models/platform/roberto_body/platform_bottom.xacro (robot description, xacro)
@@ -4,5 +4,5 @@
 	<xacro:macro name="RobertoPlatformBottom" params="name parent mesh_collis:=^|simplified mesh_visual:=^|detailed model_dir:=^">
 		<xacro:property name="ParentLink2ThisLink"> <!--parent link to this joint tf-->
-			<origin xyz="0 0 0" rpy="0 0 0"/>
+			<origin xyz="0 0 0" rpy="0 0 -${M_PI/2}"/>
 	    </xacro:property>
 	    <xacro:property name="ThisLink2Inert"> <!--this link 2 inertial center tf, mass data-->

File: src/roberto_models_jade/models/sensors/IMU/imu.xacro (robot description, xacro)
@@ -28,51 +28,57 @@
     </link>
     <xacro:property name="imu_noise_lin">
-	<noise type="tuw_advanced">
-	    <meanWhiteNoise   value="0"/>
-	    <sigmaWhiteNoise  value="0.003"/>
-	    <tauCutOff        value="${1/250}"/>
-	    <sigmaRandWalk    value="${9.8 * 0.00005}"/>
-	    <sigmaGaussMarkov value="${9.8 * 0.002}"/>
-	    <freqGaussMarkov  value="${1/100}"/>
-	</noise>
-    </xacro:property>
-    <xacro:property name="imu_noise_ang">
-	<noise type="tuw_advanced">
-	    <meanWhiteNoise   value="0"/>
-	    <sigmaWhiteNoise  value="0.00024"/>
-	    <tauCutOff        value="${1/133}"/>
-	    <sigmaRandWalk    value="${1/180 * 0.00001}"/>
-	    <sigmaGaussMarkov value="${1/180 * 0.0003}"/>
-	    <freqGaussMarkov  value="${1/40}"/>
-	</noise>
-    </xacro:property>
-    <xacro:property name="mag_noise">
-	<noise type="tuw_advanced">
-	    <meanWhiteNoise   value="0"/>
-	    <sigmaWhiteNoise  value="0.00024"/>
-	    <tauCutOff        value="${1/110}"/>
-	    <sigmaRandWalk    value="${1e-4 * 0.000006}"/>
-	    <sigmaGaussMarkov value="${1e-4 * 0.00003}"/>
-	    <freqGaussMarkov  value="${1/70}"/>
-	</noise>
+		<noise type="tuw_advanced">
+		    <meanWhiteNoise   value="0"/>
+		    <sigmaWhiteNoise  value="0.003"/>
+		    <tauCutOff        value="${1/250}"/>
+		    <sigmaRandWalk    value="${9.8 * 0.00005}"/>
+		    <sigmaGaussMarkov value="${9.8 * 0.002}"/>
+		    <freqGaussMarkov  value="${1/100}"/>
+		</noise>
+	    </xacro:property>
+	    <xacro:property name="imu_noise_ang">
+		<noise type="tuw_advanced">
+		    <meanWhiteNoise   value="0"/>
+		    <sigmaWhiteNoise  value="0.00024"/>
+		    <tauCutOff        value="${1/133}"/>
+		    <sigmaRandWalk    value="${1/180 * 0.00001}"/>
+		    <sigmaGaussMarkov value="${1/180 * 0.0003}"/>
+		    <freqGaussMarkov  value="${1/40}"/>
+		</noise>
+	    </xacro:property>
+	    <xacro:property name="mag_noise">
+		<noise type="tuw_advanced">
+		    <meanWhiteNoise   value="0"/>
+		    <sigmaWhiteNoise  value="0.00024"/>
+		    <tauCutOff        value="${1/110}"/>
+		    <sigmaRandWalk    value="${1e-4 * 0.000006}"/>
+		    <sigmaGaussMarkov value="${1e-4 * 0.00003}"/>
+		    <freqGaussMarkov  value="${1/70}"/>
+		</noise>
     </xacro:property>
     <gazebo>
-	<plugin name="gazebo_ros_imu9dof" filename="libroberto_gazebo_ros_imu9dof.so" >
-	    <rosDebugLevel>Debug</rosDebugLevel>
-	    <robotNamespace></robotNamespace>
-	    <updateRate>50.0</updateRate>
-	    <alwaysOn>true</alwaysOn>
-	    <origin xyz="${xyz}" rpy="${rpy}"/>
-	    <link_name>${name}</link_name>
-	    <imu>
-		<topic>${name}/imu</topic>
-		<angular_velocity>    <xacro:insert_block name="imu_noise_ang"/> </angular_velocity>
-		<linear_acceleration> <xacro:insert_block name="imu_noise_lin"/> </linear_acceleration>
-	    </imu>
-	    <magnetometer>
-		<topic>${name}/mag</topic>
-		<magnetic_field> <xacro:insert_block name="mag_noise"/> </magnetic_field>
-	    </magnetometer>
-	</plugin>
+		<plugin name="gazebo_ros_imu9dof" filename="libroberto_gazebo_ros_imu9dof.so" >
+		    <rosDebugLevel>Debug</rosDebugLevel>
+		    <robotNamespace></robotNamespace>
+		    <updateRate>50.0</updateRate>
+		    <alwaysOn>true</alwaysOn>
+		    <origin xyz="${xyz}" rpy="${rpy}"/>
+		    <link_name>${name}</link_name>
+		    <imu>
+				<topic>${name}/imu</topic>
+				<angular_velocity>
+					<xacro:insert_block name="imu_noise_ang"/>
+				</angular_velocity>
+				<linear_acceleration>
+					<xacro:insert_block name="imu_noise_lin"/>
+				</linear_acceleration>
+		    </imu>
+		    <magnetometer>
+				<topic>${name}/mag</topic>
+				<magnetic_field>
+					<xacro:insert_block name="mag_noise"/>
+				</magnetic_field>
+		    </magnetometer>
+		</plugin>
     </gazebo>
 </xacro:macro>
